File: doc/eagle/fm_radio.sch (EAGLE design)
At the start: 12 parts, among them J1 OLED, J2 TEA5767 module, J3 LM386 module, J4 KA2284 module

Commit message: Version 1.2-3
Parts:
- added S3: Switch_1, SparkFun-Switches:SWITCH-SPDT-SMD-AYZ0202
- S1: value Freq_Forward -> Button_2
- S2: value Freq_backward -> Button_1
Connections:
- new net N$2: S3.P, U$1.D10
- net GND: now also S3.O
- net VCC: now also S3.S
Changed lines of the file:
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@@
 <?xml version="1.0" encoding="utf-8"?>
 <!DOCTYPE eagle SYSTEM "eagle.dtd">
-<eagle version="9.1.3">
+<eagle version="9.3.0">
 <drawing>
 <settings>
@@
 <part name="U$1" library="Arduino-clone" deviceset="NANO" device=""/>
 <part name="J1" library="SparkFun-Connectors" library_urn="urn:adsk.eagle:library:513" deviceset="I2C_STANDARD" device="_NO_SILK" package3d_urn="urn:adsk.eagle:package:38094/1" value="OLED"/>
-<part name="S1" library="SparkFun-Switches" library_urn="urn:adsk.eagle:library:535" deviceset="MOMENTARY-SWITCH-SPST" device="-PTH-6.0MM" package3d_urn="urn:adsk.eagle:package:40163/1" value="Freq_Forward"/>
-<part name="S2" library="SparkFun-Switches" library_urn="urn:adsk.eagle:library:535" deviceset="MOMENTARY-SWITCH-SPST" device="-PTH-6.0MM" package3d_urn="urn:adsk.eagle:package:40163/1" value="Freq_backward"/>
+<part name="S1" library="SparkFun-Switches" library_urn="urn:adsk.eagle:library:535" deviceset="MOMENTARY-SWITCH-SPST" device="-PTH-6.0MM" package3d_urn="urn:adsk.eagle:package:40163/1" value="Button_2"/>
+<part name="S2" library="SparkFun-Switches" library_urn="urn:adsk.eagle:library:535" deviceset="MOMENTARY-SWITCH-SPST" device="-PTH-6.0MM" package3d_urn="urn:adsk.eagle:package:40163/1" value="Button_1"/>
 <part name="R1" library="eagle-ltspice" library_urn="urn:adsk.eagle:library:217" deviceset="R" device="R0603" package3d_urn="urn:adsk.eagle:package:13302/1" value="10K"/>
 <part name="R2" library="eagle-ltspice" library_urn="urn:adsk.eagle:library:217" deviceset="R" device="R0603" package3d_urn="urn:adsk.eagle:package:13302/1" value="10K"/>
@@
 <part name="SP1" library="speaker" library_urn="urn:adsk.eagle:library:365" deviceset="SMS-1308MS-2-R" device="" package3d_urn="urn:adsk.eagle:package:26519/1" value="Speaker 8ohms"/>
 <part name="SP2" library="speaker" library_urn="urn:adsk.eagle:library:365" deviceset="SMS-1308MS-2-R" device="" package3d_urn="urn:adsk.eagle:package:26519/1" value="Speaker 8 ohms"/>
+<part name="S3" library="SparkFun-Switches" library_urn="urn:adsk.eagle:library:535" deviceset="SWITCH-SPDT" device="-SMD-AYZ0202" package3d_urn="urn:adsk.eagle:package:40160/1" value="Switch_1"/>
+<part name="SUPPLY7" library="supply2" library_urn="urn:adsk.eagle:library:372" deviceset="VCC" device=""/>
 </parts>
 <sheets>
@@
 </plain>
 <instances>
-<instance part="U$1" gate="G$1" x="38.1" y="50.8"/>
-<instance part="J1" gate="G$1" x="-50.8" y="73.66"/>
-<instance part="S1" gate="G$1" x="60.96" y="63.5"/>
-<instance part="S2" gate="G$1" x="60.96" y="71.12"/>
-<instance part="R1" gate="G$1" x="-20.32" y="86.36" rot="R90"/>
-<instance part="R2" gate="G$1" x="-5.08" y="86.36" rot="R90"/>
-<instance part="J3" gate="G$1" x="-48.26" y="20.32"/>
+<instance part="U$1" gate="G$1" x="38.1" y="50.8" smashed="yes"/>
+<instance part="J1" gate="G$1" x="-50.8" y="73.66" smashed="yes">
+<attribute name="VALUE" x="-55.88" y="68.326" size="1.778" layer="96" font="vector" align="top-left"/>
+<attribute name="NAME" x="-55.88" y="81.534" size="1.778" layer="95" font="vector"/>
+</instance>
+<instance part="S1" gate="G$1" x="60.96" y="63.5" smashed="yes">
+<attribute name="NAME" x="60.96" y="65.024" size="1.778" layer="95" font="vector" align="bottom-center"/>
+<attribute name="VALUE" x="60.96" y="62.992" size="1.778" layer="96" font="vector" align="top-center"/>
+</instance>
+<instance part="S2" gate="G$1" x="60.96" y="71.12" smashed="yes">
+<attribute name="NAME" x="60.96" y="72.644" size="1.778" layer="95" font="vector" align="bottom-center"/>
+<attribute name="VALUE" x="60.96" y="70.612" size="1.778" layer="96" font="vector" align="top-center"/>
+</instance>
+<instance part="R1" gate="G$1" x="-20.32" y="86.36" smashed="yes" rot="R90">
+<attribute name="NAME" x="-21.8186" y="82.55" size="1.778" layer="95" rot="R90"/>
+<attribute name="VALUE" x="-17.018" y="82.55" size="1.778" layer="96" rot="R90"/>
+</instance>
+<instance part="R2" gate="G$1" x="-5.08" y="86.36" smashed="yes" rot="R90">
+<attribute name="NAME" x="-6.5786" y="82.55" size="1.778" layer="95" rot="R90"/>
+<attribute name="VALUE" x="-1.778" y="82.55" size="1.778" layer="96" rot="R90"/>
+</instance>
+<instance part="J3" gate="G$1" x="-48.26" y="20.32" smashed="yes">
+<attribute name="VALUE" x="-53.34" y="10.414" size="1.778" layer="96" font="vector"/>
+<attribute name="NAME" x="-53.34" y="30.988" size="1.778" layer="95" font="vector"/>
+</instance>
 <instance part="J2" gate="G$1" x="-48.26" y="50.8" smashed="yes">
 <attribute name="VALUE" x="-53.34" y="40.894" size="1.778" layer="96" font="vector"/>
 <attribute name="NAME" x="-53.34" y="61.468" size="1.778" layer="95" font="vector"/>
 </instance>
-<instance part="J4" gate="G$1" x="-48.26" y="-5.08"/>
-<instance part="SUPPLY1" gate="G$1" x="-12.7" y="99.06"/>
-<instance part="SUPPLY2" gate="GND" x="71.12" y="58.42"/>
-<instance part="SUPPLY3" gate="GND" x="10.16" y="27.94"/>
-<instance part="SUPPLY4" gate="G$1" x="0" y="38.1" rot="R90"/>
-<instance part="SUPPLY5" gate="G$1" x="-22.86" y="73.66" rot="R270"/>
-<instance part="SUPPLY6" gate="GND" x="-35.56" y="66.04"/>
-<instance part="ANT1" gate="A" x="-71.12" y="40.64"/>
-<instance part="SP1" gate="A" x="10.16" y="0" rot="R270"/>
-<instance part="SP2" gate="A" x="43.18" y="0" rot="R270"/>
+<instance part="J4" gate="G$1" x="-48.26" y="-5.08" smashed="yes">
+<attribute name="VALUE" x="-53.34" y="-14.986" size="1.778" layer="96" font="vector"/>
+<attribute name="NAME" x="-53.34" y="5.588" size="1.778" layer="95" font="vector"/>
+</instance>
+<instance part="SUPPLY1" gate="G$1" x="-12.7" y="99.06" smashed="yes">
+<attribute name="VALUE" x="-14.605" y="102.235" size="1.778" layer="96"/>
+</instance>
+<instance part="SUPPLY2" gate="GND" x="73.66" y="55.88" smashed="yes" rot="R90">
+<attribute name="VALUE" x="76.835" y="53.975" size="1.778" layer="96" rot="R90"/>
+</instance>
+<instance part="SUPPLY3" gate="GND" x="10.16" y="27.94" smashed="yes">
+<attribute name="VALUE" x="8.255" y="24.765" size="1.778" layer="96"/>
+</instance>
+<instance part="SUPPLY4" gate="G$1" x="0" y="38.1" smashed="yes" rot="R90">
+<attribute name="VALUE" x="-3.175" y="36.195" size="1.778" layer="96" rot="R90"/>
+</instance>
+<instance part="SUPPLY5" gate="G$1" x="-22.86" y="73.66" smashed="yes" rot="R270">
+<attribute name="VALUE" x="-19.685" y="75.565" size="1.778" layer="96" rot="R270"/>
+</instance>
+<instance part="SUPPLY6" gate="GND" x="-35.56" y="66.04" smashed="yes">
+<attribute name="VALUE" x="-37.465" y="62.865" size="1.778" layer="96"/>
+</instance>
+<instance part="ANT1" gate="A" x="-71.12" y="40.64" smashed="yes">
+<attribute name="NAME" x="-73.66" y="41.91" size="1.778" layer="95"/>
+<attribute name="VALUE" x="-68.58" y="35.56" size="1.778" layer="96"/>
+</instance>
+<instance part="SP1" gate="A" x="10.16" y="0" smashed="yes" rot="R270">
+<attribute name="NAME" x="11.43" y="-5.08" size="1.778" layer="95" rot="R270"/>
+<attribute name="VALUE" x="7.62" y="-5.08" size="1.778" layer="96" rot="R270"/>
+</instance>
+<instance part="SP2" gate="A" x="43.18" y="0" smashed="yes" rot="R270">
+<attribute name="NAME" x="44.45" y="-5.08" size="1.778" layer="95" rot="R270"/>
+<attribute name="VALUE" x="40.64" y="-5.08" size="1.778" layer="96" rot="R270"/>
+</instance>
+<instance part="S3" gate="1" x="63.5" y="40.64" smashed="yes">
+<attribute name="NAME" x="64.77" y="43.688" size="1.778" layer="95" font="vector" align="bottom-center"/>
+<attribute name="VALUE" x="64.516" y="37.338" size="1.778" layer="96" font="vector" align="top-center"/>
+</instance>
+<instance part="SUPPLY7" gate="G$1" x="73.66" y="33.02" smashed="yes" rot="R270">
+<attribute name="VALUE" x="76.835" y="34.925" size="1.778" layer="96" rot="R270"/>
+</instance>
 </instances>
 <busses>
@@
 <junction x="-27.94" y="73.66"/>
 </segment>
+<segment>
+<pinref part="S3" gate="1" pin="S"/>
+<wire x1="68.58" y1="38.1" x2="71.12" y2="38.1" width="0.1524" layer="91"/>
+<wire x1="71.12" y1="38.1" x2="71.12" y2="33.02" width="0.1524" layer="91"/>
+<pinref part="SUPPLY7" gate="G$1" pin="VCC"/>
+</segment>
 </net>
 <net name="SDA" class="0">
@@
 <wire x1="71.12" y1="63.5" x2="66.04" y2="63.5" width="0.1524" layer="91"/>
 <pinref part="SUPPLY2" gate="GND" pin="GND"/>
-<wire x1="71.12" y1="63.5" x2="71.12" y2="60.96" width="0.1524" layer="91"/>
+<wire x1="71.12" y1="63.5" x2="71.12" y2="55.88" width="0.1524" layer="91"/>
 <junction x="71.12" y="63.5"/>
+<pinref part="S3" gate="1" pin="O"/>
+<wire x1="68.58" y1="43.18" x2="71.12" y2="43.18" width="0.1524" layer="91"/>
+<wire x1="71.12" y1="43.18" x2="71.12" y2="55.88" width="0.1524" layer="91"/>
+<junction x="71.12" y="55.88"/>
 </segment>
 <segment>
@@
 </segment>
 </net>
+<net name="N$2" class="0">
+<segment>
+<wire x1="53.34" y1="58.42" x2="58.42" y2="58.42" width="0.1524" layer="91"/>
+<wire x1="58.42" y1="58.42" x2="58.42" y2="40.64" width="0.1524" layer="91"/>
+<pinref part="S3" gate="1" pin="P"/>
+<wire x1="58.42" y1="40.64" x2="60.96" y2="40.64" width="0.1524" layer="91"/>
+<pinref part="U$1" gate="G$1" pin="D10"/>
+<wire x1="48.26" y1="60.96" x2="53.34" y2="60.96" width="0.1524" layer="91"/>
+<wire x1="53.34" y1="60.96" x2="53.34" y2="58.42" width="0.1524" layer="91"/>
+</segment>
+</net>
